Commit message: (fix) fix no contact force in isaac gym, fix feet in air

File: resources/robots/b2/urdf/b2.urdf (robot description, URDF)
Before this commit: robot b2_description, 44 links, 43 joints
Links:
- added link gripperMover, mass 0.27621302; collision mesh filename=../dae/z1_GripperMover.dae scale=1 1 1; visual mesh filename=../dae/z1_GripperMover.dae scale=1 1 1
- added link gripperStator, mass 0.52603655; collision mesh filename=../dae/z1_GripperStator.dae scale=1 1 1; visual mesh filename=../dae/z1_GripperStator.dae scale=1 1 1
Joints:
- added joint gripperStator: type fixed, parent link06, child gripperStator, origin xyz=0.051 0.0 0.0 rpy=0 0 0
- added joint jointGripper: type fixed, parent gripperStator, child gripperMover, origin xyz=0.049 0.0 0 rpy=0 0 0, axis 0 1 0, limit lower=-1.57 upper=0.0 effort=30.0 velocity=10
